File: serverAnywhere/serverAnywhere.kicad_sch (KiCad schematic)
At the start: 0 parts

Commit message: Hopefully finished
Parts:
- added J1: USB_C_Receptacle_PowerOnly_6P, Connector_USB:USB_C_Receptacle_GCT_USB4125-xx-x-0190_6P_TopMnt_Horizontal, symbol Connector:USB_C_Receptacle_PowerOnly_6P
- added J2: USB_C_Receptacle_USB2.0_14P, Connector_USB:USB_C_Receptacle_GCT_USB4105-xx-A_16P_TopMnt_Horizontal, symbol Connector:USB_C_Receptacle_USB2.0_14P
- added R1, R2: 5k1, Resistor_SMD:R_0805_2012Metric_Pad1.20x1.40mm_HandSolder, symbol Device:R_Small
- added U1: USBLC6-2SC6, Package_TO_SOT_SMD:SOT-23-6, symbol Power_Protection:USBLC6-2SC6
Connections:
- new net: J2.A5 (CC1), R2.1
- new net: J2.A4 (VBUS), J2.A9 (VBUS), J2.B4 (VBUS), J2.B9 (VBUS)
- new net: J2.B5 (CC2), R1.1
- new net +5V: J1.A9 (VBUS), J1.B9 (VBUS)
- new net CC1: J1.B5 (CC2)
- new net CC2: J1.A5 (CC1)
- new net GND: J1.A12 (GND), J1.B12 (GND), J1.S1 (SHIELD), J2.A1 (GND), J2.A12 (GND), J2.B1 (GND), J2.B12 (GND), J2.S1 (SHIELD), R1.2, R2.2, U1.2 (GND)
- new net HighSpeed/USB_N: U1.4 (I/O2)
- new net HighSpeed/USB_P: U1.3 (I/O2)
- new net USB_N: J2.A7 (D-), J2.B7 (D-), U1.6 (I/O1)
- new net USB_P: J2.A6 (D+), J2.B6 (D+), U1.1 (I/O1)
- no-connect marks 0 -> 2
Other:
- added sheet HighSpeed (highspeed.kicad_sch)
- added sheet Misc (misc.kicad_sch)
